Commit message: Sliding Mode Control scripts added

File: src/sawyer_robot/sawyer_description/urdf/right_eraser_force_torque_gazebo.urdf.xacro (robot description, xacro)
@@ -13,5 +13,5 @@
   <xacro:include filename="$(find sensor_description)/urdf/ft_sensor_ati.urdf.xacro"/>
   <xacro:ft_sensor_ft45 parent="right_plate_sensor" name="right" type="ft45">
-    <origin xyz="0 0 0" rpy="0 0 0"/>
+    <origin xyz="0 0 0" rpy="0 0 ${M_PI/2}"/>
   </xacro:ft_sensor_ft45>
   <xacro:include filename="$(find intera_tools_description)/urdf/plate/plate.xacro" />
